Commit message: friction+centre of mass fixed

File: ros2_ws/src/main/urdf/materials.xacro (robot description, xacro)
@@ -1,6 +1,12 @@
 <?xml version="1.0" ?>
 <robot name="Rover" xmlns:xacro="http://www.ros.org/wiki/xacro" >
-<material name="silver">
+<material name="_silver">
   <color rgba="0.700 0.700 0.700 1.000"/>
 </material>
+<material name="blue">
+  <color rgba="0.0 0.0 1.0 1.0" />
+</material>
+<material name="dark">
+  <color rgba="0.0 0.0 1.0 1.0" />
+</material>
 </robot>

File: ros2_ws/src/main/urdf/rover.xacro (robot description, xacro)
@@ -1,144 +1,154 @@
-<?xml version="1.0" ?>
+<?xml version="1.0"?>
 <robot name="Rover" xmlns:xacro="http://www.ros.org/wiki/xacro">
-<xacro:include filename="$(find main)/urdf/materials.xacro" />
-<xacro:include filename="$(find main)/urdf/Rover.trans" />
-<xacro:include filename="$(find main)/urdf/Rover.gazebo" />
-<xacro:include filename="spring.xacro"/>
-<!-- <link name="dummy_base_link"></link> -->
-<link name="base_link">
-  <inertial>
-    <origin xyz="-6.106915349179497e-13 -0.02576797376370591 0.3408721287496551" rpy="0 0 -1.57"/>
-    <mass value="119.00094541166615"/>
-    <inertia ixx="11.367893" iyy="2.895706" izz="13.361019" ixy="-0.0" iyz="0.11269" ixz="-0.0"/>
-  </inertial>
-  <visual>
-    <origin xyz="0 0 0" rpy="0 0 1.57"/>
-    <geometry>
-      <mesh filename="file://$(find main)/meshes/base_link.stl" scale="0.001 0.001 0.001"/>
-    </geometry>
-    <material name="ok">
-      <color rgba="0.4 0.4 0.4 1.0"/>
-    </material>
-  </visual>
-  <collision>
-    <origin xyz="0 0 0" rpy="0 0 1.57"/>
-    <geometry>
-      <mesh filename="file://$(find main)/meshes/base_link.stl" scale="0.001 0.001 0.001"/>
-    </geometry>
-  </collision>
-</link>
-<link name="fr_wheel_1"><xacro:wheel/></link>
-<link name="mr_wheel_1"><xacro:wheel/></link>
-<link name="br_wheel_1"><xacro:wheel/></link>
-<link name="fl_wheel_1"><xacro:left_wheel/></link>
-<link name="ml_wheel_1"><xacro:left_wheel/></link>
-<link name="bl_wheel_1"><xacro:left_wheel/></link>
-<link name="cam_link_1">
-  <visual>
-    <origin xyz="0 0 0" rpy="0 0 0"/>
-    <geometry>
-      <cylinder radius="0.01" length="0.2"/>
-      <!-- <mesh filename="file://$(find main)/meshes/cam_link_1.stl" scale="0.001 0.001 0.001"/> -->
-    </geometry>
-    <material name="silver"/>
-  </visual>
-</link>
-<link name="cam_1">
-  <visual>
-    <origin xyz="0 0 0" rpy="0 0 0"/>
-    <geometry>
-      <box size="0.03 0.1 0.03"/>
-    </geometry>
-    <material name="silver">
-    </material>
-  </visual>
-</link>
-<link name="rgbd_1">
-</link>
-<gazebo reference="base_link">
-  <sensor name="imu" type="imu">
-    <always_on>true</always_on>
-    <!-- <visualize>true</visualize> -->
-    <update_rate>20</update_rate>
-    <gz_frame_id>odom</gz_frame_id>
-    <child_frame_id>base_link</child_frame_id>
-    <topic>imu</topic>
-  </sensor>
-</gazebo>
-<gazebo reference="rgbd_1">
-  <sensor name="depth_camera" type="depth">
-    <always_on>true</always_on>
-    <!-- <visualize>true</visualize> -->
-    <update_rate>20</update_rate>
-    <topic>depth_camera/image</topic>
-    <gz_frame_id>rgbd_1</gz_frame_id>
-    <camera name="depth_camera">
-      <camera_info_topic>depth_camera/camera_info</camera_info_topic>
-      <horizontal_fov>1.8</horizontal_fov>
-      <image>
-        <width>640</width>
-        <height>640</height>
-      </image>
-      <clip>
-        <near>0.5</near>
-        <far>25</far>
-      </clip>
-    </camera>
-  </sensor>
-</gazebo>
-<gazebo reference="cam_1">
-  <sensor name="camera" type="camera">
-    <always_on>true</always_on>
-    <visualize>true</visualize>
-    <update_rate>20</update_rate>
-    <topic>camera/image</topic>
-    <gz_frame_id>cam_1</gz_frame_id>
-    <camera name="camera">
-      <camera_info_topic>camera/camera_info</camera_info_topic>
-      <horizontal_fov>1.8</horizontal_fov>
-      <image>
-        <width>640</width>
-        <height>640</height>
-      </image>
-      <clip>
-        <near>0.5</near>
-        <far>50</far>
-      </clip>
-    </camera>
-  </sensor>
-</gazebo>
-<gazebo reference="base_link">
-  <sensor name="gps" type="gps">
-  <always_on>true</always_on>
-  <update_rate>20</update_rate>
-  <visualize>true</visualize>
-  <pose>0 0 0 0 0 0</pose>
-  <topic>gps</topic>
-  <gz_frame_id>base_link</gz_frame_id>
-  <!-- <child_frame_id>base_link</child_frame_id> -->
-  <gps>
-    <position_sensing>
-      <horizontal>
-        <noise type="gaussian">
-          <mean>0.0</mean>
-          <stddev>0.0</stddev>
-        </noise>
-      </horizontal>
-      <vertical>
-        <noise type="gaussian">
-          <mean>0.0</mean>
-          <stddev>0.0</stddev>
-        </noise>
-      </vertical>
-    </position_sensing>
-  </gps>
-  <!-- <plugin name="my_gps_plugin" filename="libgazebo_ros_gps_sensor.so">
+  <xacro:include filename="$(find main)/urdf/materials.xacro" />
+  <xacro:include filename="$(find main)/urdf/Rover.trans" />
+  <xacro:include filename="$(find main)/urdf/Rover.gazebo" />
+  <xacro:include filename="$(find main)/urdf/spring.xacro" />
+  <!-- <link name="dummy_base_link"></link> -->
+  <link name="base_link">
+    <inertial>
+      <origin xyz="0.0 0.0 0.3" rpy="0 0 -1.57" />
+      <mass value="40.0" />
+      <inertia ixx="11.367893" iyy="2.895706" izz="13.361019" ixy="0.0" iyz="0.0" ixz="0.0" />
+    </inertial>
+    <visual>
+      <origin xyz="0 0 0" rpy="0 0 1.57" />
+      <geometry>
+        <mesh filename="file://$(find main)/meshes/base_link.stl" scale="0.001 0.001 0.001" />
+      </geometry>
+      <material name="_silver" />
+    </visual>
+    <collision>
+      <origin xyz="0 0 0" rpy="0 0 1.57" />
+      <geometry>
+        <mesh filename="file://$(find main)/meshes/base_link.stl" scale="0.001 0.001 0.001" />
+      </geometry>
+    </collision>
+  </link>
+  <link name="fr_wheel_1">
+    <xacro:wheel />
+  </link>
+  <link name="mr_wheel_1">
+    <xacro:wheel />
+  </link>
+  <link name="br_wheel_1">
+    <xacro:wheel />
+  </link>
+  <link name="fl_wheel_1">
+    <xacro:left_wheel />
+  </link>
+  <link name="ml_wheel_1">
+    <xacro:left_wheel />
+  </link>
+  <link name="bl_wheel_1">
+    <xacro:left_wheel />
+  </link>
+  <link name="cam_link_1">
+    <visual>
+      <origin xyz="0 0 0" rpy="0 0 0" />
+      <geometry>
+        <cylinder radius="0.01" length="0.2" />
+        <!-- <mesh filename="file://$(find main)/meshes/cam_link_1.stl" scale="0.001 0.001 0.001"/> -->
+      </geometry>
+      <material name="dark" />
+    </visual>
+  </link>
+  <link name="cam_1">
+    <visual>
+      <origin xyz="0 0 0" rpy="0 0 0" />
+      <geometry>
+        <box size="0.03 0.1 0.03" />
+      </geometry>
+      <material name="dark">
+      </material>
+    </visual>
+  </link>
+  <link name="rgbd_1">
+  </link>
+  <gazebo reference="base_link">
+    <sensor name="imu" type="imu">
+      <always_on>true</always_on>
+      <!-- <visualize>true</visualize> -->
+      <update_rate>20</update_rate>
+      <gz_frame_id>odom</gz_frame_id>
+      <child_frame_id>base_link</child_frame_id>
+      <topic>imu</topic>
+    </sensor>
+  </gazebo>
+  <gazebo reference="rgbd_1">
+    <sensor name="depth_camera" type="depth">
+      <always_on>true</always_on>
+      <!-- <visualize>true</visualize> -->
+      <update_rate>20</update_rate>
+      <topic>depth_camera/image</topic>
+      <gz_frame_id>rgbd_1</gz_frame_id>
+      <camera name="depth_camera">
+        <camera_info_topic>depth_camera/camera_info</camera_info_topic>
+        <horizontal_fov>1.8</horizontal_fov>
+        <image>
+          <width>640</width>
+          <height>640</height>
+        </image>
+        <clip>
+          <near>0.5</near>
+          <far>25</far>
+        </clip>
+      </camera>
+    </sensor>
+  </gazebo>
+  <gazebo reference="cam_1">
+    <sensor name="camera" type="camera">
+      <always_on>true</always_on>
+      <visualize>true</visualize>
+      <update_rate>20</update_rate>
+      <topic>camera/image</topic>
+      <gz_frame_id>cam_1</gz_frame_id>
+      <camera name="camera">
+        <camera_info_topic>camera/camera_info</camera_info_topic>
+        <horizontal_fov>1.8</horizontal_fov>
+        <image>
+          <width>640</width>
+          <height>640</height>
+        </image>
+        <clip>
+          <near>0.5</near>
+          <far>50</far>
+        </clip>
+      </camera>
+    </sensor>
+  </gazebo>
+  <gazebo reference="base_link">
+    <sensor name="gps" type="gps">
+      <always_on>true</always_on>
+      <update_rate>20</update_rate>
+      <visualize>true</visualize>
+      <pose>0 0 0 0 0 0</pose>
+      <topic>gps</topic>
+      <gz_frame_id>base_link</gz_frame_id>
+      <!-- <child_frame_id>base_link</child_frame_id> -->
+      <gps>
+        <position_sensing>
+          <horizontal>
+            <noise type="gaussian">
+              <mean>0.0</mean>
+              <stddev>0.0</stddev>
+            </noise>
+          </horizontal>
+          <vertical>
+            <noise type="gaussian">
+              <mean>0.0</mean>
+              <stddev>0.0</stddev>
+            </noise>
+          </vertical>
+        </position_sensing>
+      </gps>
+      <!-- <plugin name="my_gps_plugin" filename="libgazebo_ros_gps_sensor.so">
     <ros>
       <remapping>~/out:=/gps/fix</remapping>
     </ros>
   </plugin> -->
-</sensor>
-</gazebo>
-<!--
+    </sensor>
+  </gazebo>
+  <!--
 <joint name="dummy" type="fixed">
   <origin xyz="0 0 0" rpy="0 0 0"/>
@@ -146,113 +156,54 @@
   <child link="base_link"/>
 </joint> -->
-<link name="spring_fr">
-  <xacro:spring_link/>
-</link>
-<joint name="fr_spring_to_body" type="prismatic">
-  <origin xyz="0.491042 -0.35  0.196191" rpy="0 0 0 "/>
-  <parent link="base_link"/>
-  <child link="spring_fr"/>
-  <xacro:spring_joint/>
-  <sensor name="force_torque" type="force_torque">
-          <update_rate>30</update_rate>
-          <visualize>true</visualize>
-          <topic>force</topic>
-        </sensor>
-  </joint>
-<joint name="frw_to_body" type="continuous">
-  <origin xyz="0.0 0.0 0.0" rpy="0 0 -1.57"/>
-  <parent link="spring_fr"/>
-  <child link="fr_wheel_1"/>
-  <axis xyz="-1.0 0.0 0.0"/>
-</joint>
-<link name="spring_mr">
-  <xacro:spring_link/>
-</link>
-<joint name="mr_spring_to_body" type="prismatic">
-  <origin xyz="0.051042 -0.35  0.196191" rpy="0 0 0 "/>
-  <parent link="base_link"/>
-  <child link="spring_mr"/>
-  <xacro:spring_joint/>
-</joint>
-<joint name="mrw_to_body" type="continuous">
-  <origin xyz="0.0 0.0 0.0" rpy="0 0 -1.57"/>
-  <parent link="spring_mr"/>
-  <child link="mr_wheel_1"/>
-  <axis xyz="-1.0 0.0 0.0"/>
-</joint>
-<link name="spring_br">
-  <xacro:spring_link/>
-</link>
-<joint name="br_spring_to_body" type="prismatic">
-  <origin xyz="-0.388958 -0.35  0.196191" rpy="0 0 0 "/>
-  <parent link="base_link"/>
-  <child link="spring_br"/>
-  <xacro:spring_joint/>
-</joint>
-<joint name="brw_to_body" type="continuous">
-  <origin xyz="0.0 0.0 0.0" rpy="0 0 -1.57"/>
-  <parent link="spring_br"/>
-  <child link="br_wheel_1"/>
-  <axis xyz="-1.0 0.0 0.0"/>
-</joint>
-<link name="spring_fl">
-  <xacro:spring_link/>
-</link>
-<joint name="fl_spring_to_body" type="prismatic">
-  <origin xyz="0.491042 0.35  0.196191" rpy="0 0 0 "/>
-  <parent link="base_link"/>
-  <child link="spring_fl"/>
-  <xacro:spring_joint/>
-</joint>
-<joint name="flw_to_body" type="continuous">
-  <origin xyz="0.0 0.0 0.0" rpy="0 0 -1.57"/>
-  <parent link="spring_fl"/>
-  <child link="fl_wheel_1"/>
-  <axis xyz="-1.0 0.0 0.0"/>
-</joint>
-<link name="spring_ml">
-  <xacro:spring_link/>
-</link>
-<joint name="ml_spring_to_body" type="prismatic">
-  <origin xyz="0.051042 0.35  0.196191" rpy="0 0 0 "/>
-  <parent link="base_link"/>
-  <child link="spring_ml"/>
-  <xacro:spring_joint/>
-</joint>
-<joint name="mlw_to_body" type="continuous">
-  <origin xyz="0.0 0.0 0.0" rpy="0 0 -1.57"/>
-  <parent link="spring_ml"/>
-  <child link="ml_wheel_1"/>
-  <axis xyz="-1.0 0.0 0.0"/>
-</joint>
-<link name="spring_bl">
-  <xacro:spring_link/>
-</link>
-<joint name="bl_spring_to_body" type="prismatic">
-  <origin xyz="-0.388958 0.35 0.196191" rpy="0 0 0 "/>
-  <parent link="base_link"/>
-  <child link="spring_bl"/>
-  <xacro:spring_joint/>
-</joint>
-<joint name="blw_to_body" type="continuous">
-  <origin xyz="0.0 0.0 0.0" rpy="0 0 -1.57"/>
-  <parent link="spring_bl"/>
-  <child link="bl_wheel_1"/>
-  <axis xyz="-1.0 0.0 0.0"/>
-</joint>
-<joint name="camlink_to_body" type="fixed">
-  <origin xyz="0.6 0.0001 0.5" rpy="0 0 0"/>
-  <parent link="base_link"/>
-  <child link="cam_link_1"/>
-</joint>
-<joint name="cam_to_camlink" type="fixed">
-  <origin xyz="0 0 0.1" rpy="0 0.60 0"/>
-  <parent link="cam_link_1"/>
-  <child link="cam_1"/>
-</joint>
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
File: ros2_ws/src/main/urdf/spring.xacro (robot description, xacro)
@@ -1,71 +1,87 @@
 <?xml version="1.0"?>
-<robot xmlns:xacro="http://www.ros.org/wiki/xacro" >
+<robot xmlns:xacro="http://www.ros.org/wiki/xacro">
+    <!-- <xacro:include filename="$(find main)/urdf/materials.xacro" /> -->
     <xacro:macro name="spring_link">
         <inertial>
-            <origin xyz="0.0 0.0  0.0 " rpy="0 0 0"/>
-            <mass value="0.01"/>
-            <inertia ixx="0.0" iyy="0.0" izz="0.0" ixy="0.0" iyz="0.0" ixz="0.0"/>
+            <origin xyz="0.0 0.0  0.0 " rpy="0 0 0" />
+            <mass value="0.01" />
+            <inertia ixx="0.0" iyy="0.0" izz="0.0" ixy="0.0" iyz="0.0" ixz="0.0" />
         </inertial>
         <visual>
-            <origin xyz="0 0 0" rpy="0 0 0"/>
+            <origin xyz="0 0 0" rpy="0 0 0" />
             <geometry>
-            <box size="0.1 0.1 0.1"/>
+                <box size="0.1 0.1 0.1" />
             </geometry>
-            <material name="silver">
-            </material>
         </visual>
     </xacro:macro>
     <xacro:macro name="spring_joint">
-        <axis xyz="0.0 0.0 -1.0"/>
-            <limit lower="-0.050" upper="0.050"  velocity="-1.0" effort="-1.0"/>
-            <dynamics damping="50.0" spring_reference ="0.0" spring_stiffness="5.0"/>
-            <ode>
-                <fudge_factor>0.1</fudge_factor>
-                <cfm>0.00001</cfm>
-                <erp>0.8</erp>
-            </ode>
+        <axis xyz="0.0 0.0 0.0" />
+        <limit lower="0.0" upper="0.0" velocity="0.0" effort="-1.0" />
+    </xacro:macro>
+    <xacro:macro name="surface">
+        <surface>
+            <friction>
+                <ode>
+                    <mu>1</mu>
+                    <mu2>1</mu2>
+                    <slip1>0.01</slip1>
+                    <slip2>0.01</slip2>
+                </ode>
+            </friction>
+            <contact>
+                <ode>
+                    <soft_cfm>0</soft_cfm>
+                    <soft_erp>0.2</soft_erp>
+                    <kp>1e+13</kp>
+                    <kd>1</kd>
+                    <max_vel>0.01</max_vel>
+                    <min_depth>0.0</min_depth>
+                </ode>
+            </contact>
+        </surface>
     </xacro:macro>
     <xacro:macro name="wheel">
-    <inertial>
-            <origin xyz="0.05 0 0" rpy="0 1.57 0"/>
-            <mass value="11.6"/>
-            <inertia  ixx="0.124" ixy = "0" ixz = "0"
-              iyy="0.124" iyz = "0"
-              izz="0.21"/>
-            </inertial>
-            <visual>
-            <origin xyz="0.05 0 0" rpy="0 1.57 0"/>
+        <inertial>
+            <origin xyz="0.05 0 0" rpy="0 1.5707 0" />
+            <mass value="11.6" />
+            <inertia ixx="0.124" ixy="0" ixz="0"
+                iyy="0.124" iyz="0"
+                izz="0.21" />
+        </inertial>
+        <visual>
+            <origin xyz="0.05 0 0" rpy="0 1.5707 0" />
             <geometry>
-                <cylinder radius="0.19" length="0.14"/>
+                <cylinder radius="0.19" length="0.14" />
             </geometry>
-            <material name="blue"/>
-            </visual>
-            <collision>
-                <origin xyz="0.05 0 0" rpy="0 1.57 0"/>
-                    <geometry>
-                <cylinder radius="0.19" length="0.14"/>
-                </geometry>
+        </visual>
+        <collision>
+            <origin xyz="0.05 0 0" rpy="0 1.5707 0" />
+            <geometry>
+                <cylinder radius="0.19" length="0.14" />
+            </geometry>
+            <xacro:surface />
         </collision>
     </xacro:macro>
     <xacro:macro name="left_wheel">
-            <inertial>
-            <origin xyz="-0.05 0 0" rpy="0 1.57 3.14"/>
-            <mass value="11.6"/>
-            <inertia  ixx="0.124" ixy = "0" ixz = "0"
-              iyy="0.124" iyz = "0"
-              izz="0.21"/>
-            </inertial>
-            <visual>
-            <origin xyz="-0.05 0 0" rpy="0 1.57 3.14"/>
+        <inertial>
+            <origin xyz="-0.05 0 0" rpy="0 1.5707 3.1415" />
+            <mass value="11.6" />
+            <inertia ixx="0.124" ixy="0" ixz="0"
+                iyy="0.124" iyz="0"
+                izz="0.21" />
+        </inertial>
+        <visual>
+            <origin xyz="-0.050 0 0" rpy="0 1.5707 3.1415" />
             <geometry>
-                <cylinder radius="0.19" length="0.14"/>
+                <cylinder radius="0.19" length="0.14" />
             </geometry>
-            <material name="blue"/>
-            </visual>
-            <collision>
-                <origin xyz="-0.05 0 0" rpy="0 1.57 3.14"/>
-                    <geometry>
-                <cylinder radius="0.19" length="0.14"/>
-                </geometry>
+            <material name="blue" />
+        </visual>
+        <collision>
+            <origin xyz="-0.05 0 0" rpy="0 1.57 3.1415" />
+            <geometry>
+                <cylinder radius="0.19" length="0.14" />
+            </geometry>
+            <xacro:surface />
         </collision>
     </xacro:macro>
