Commit message: some project structure added

File: ros2_ws/src/main/urdf/rover.xacro (robot description, xacro)
@@ -4,5 +4,5 @@
 <xacro:include filename="$(find main)/urdf/Rover.trans" />
 <xacro:include filename="$(find main)/urdf/Rover.gazebo" />
-<link name="dummy_base_link"></link>
+<!-- <link name="dummy_base_link"></link> -->
 <link name="base_link">
   <inertial>
@@ -197,5 +197,5 @@
     <always_on>true</always_on>
     <visualize>true</visualize>
-    <update_rate>10</update_rate>
+    <update_rate>20</update_rate>
     <topic>depth_camera/image</topic>
     <gz_frame_id>cam_1</gz_frame_id>
@@ -214,9 +214,10 @@
   </sensor>
 </gazebo>
+<!--
 <joint name="dummy" type="fixed">
-  <origin xyz="0.0 0.0 0.0" rpy="0 0 0"/>
+  <origin xyz="0 0 0" rpy="0 0 0"/>
   <parent link="dummy_base_link"/>
   <child link="base_link"/>
-</joint>
+</joint> -->
 <joint name="frw_to_body" type="continuous">
   <origin xyz="0.491042 -0.35  0.196191" rpy="0 0 -1.57"/>

Commit message: gps beta + nav2 working(stupid)

File: ros2_ws/src/main/urdf/rover.xacro (robot description, xacro)
@@ -214,4 +214,35 @@
   </sensor>
 </gazebo>
+<gazebo reference="cam_1">
+  <sensor name="tb3_gps" type="navsat">
+  <always_on>true</always_on>
+  <update_rate>10</update_rate>
+  <visualize>true</visualize>
+  <pose>0 0 0 0 0 0</pose>
+  <topic>gps</topic>
+  <gz_frame_id>cam_1</gz_frame_id>
+  <gps>
+    <position_sensing>
+      <horizontal>
+        <noise type="gaussian">
+          <mean>0.0</mean>
+          <stddev>0.00001</stddev>
+        </noise>
+      </horizontal>
+      <vertical>
+        <noise type="gaussian">
+          <mean>0.0</mean>
+          <stddev>0.00001</stddev>
+        </noise>
+      </vertical>
+    </position_sensing>
+  </gps>
+  <!-- <plugin name="my_gps_plugin" filename="libgazebo_ros_gps_sensor.so">
+    <ros>
+      <remapping>~/out:=/gps/fix</remapping>
+    </ros>
+  </plugin> -->
+</sensor>
+</gazebo>
 <!--
 <joint name="dummy" type="fixed">
@@ -257,5 +288,5 @@
 </joint>
 <joint name="camlink_to_body" type="fixed">
-  <origin xyz="0.6 0 0.5" rpy="0 0 0"/>
+  <origin xyz="0.6 0.0001 0.5" rpy="0 0 0"/>
   <parent link="base_link"/>
   <child link="cam_link_1"/>

Commit message: Povestka_beta

File: ros2_ws/src/main/urdf/rover.xacro (robot description, xacro)
@@ -251,37 +251,175 @@
   <child link="base_link"/>
 </joint> -->
+<link name="spring_fr">
+  <inertial>
+    <origin xyz="0.00005 0.00005  0.00005 " rpy="0 0 0"/>
+    <mass value="0.01"/>
+    <inertia ixx="0.0000006" iyy="0.0000006" izz="0.0000006" ixy="0.0" iyz="0.0" ixz="0.0"/>
+  </inertial>
+  <visual>
+    <origin xyz="0 0 0" rpy="0 0 0"/>
+    <geometry>
+      <box size="0.010 0.010 0.010"/>
+    </geometry>
+    <material name="silver">
+    </material>
+  </visual>
+</link>
+<joint name="fr_spring_to_body" type="prismatic">
+  <origin xyz="0.491042 -0.35  0.196191" rpy="0 0 0 "/>
+  <parent link="base_link"/>
+  <child link="spring_fr"/>
+  <axis xyz="0.0 0.0 1.0"/>
+  <limit lower="-0.05" upper="0.05" velocity="1.0" effort="10.0" />
+  <dynamics damping="500.0" spring_reference = "0.0" spring_stiffness = "10000.1" friction = "0.75"/>
+</joint>
 <joint name="frw_to_body" type="continuous">
-  <origin xyz="0.491042 -0.35  0.196191" rpy="0 0 -1.57"/>
-  <parent link="base_link"/>
+  <origin xyz="0.0 0.0 0.0" rpy="0 0 -1.57"/>
+  <parent link="spring_fr"/>
   <child link="fr_wheel_1"/>
   <axis xyz="-1.0 0.0 0.0"/>
 </joint>
+<link name="spring_mr">
+  <inertial>
+    <origin xyz="0.0000000000000005 0.00000000000000000005 0.00000000000000000005" rpy="0 0 0"/>
+    <mass value="0.00000000000001"/>
+    <inertia ixx="0.0000006" iyy="0.0000006" izz="0.0000006" ixy="0.0" iyz="0.0" ixz="0.0"/>
+  </inertial>
+  <visual>
+    <origin xyz="0 0 0" rpy="0 0 0"/>
+    <geometry>
+      <box size="0.010 0.010 0.010"/>
+    </geometry>
+    <material name="silver">
+    </material>
+  </visual>
+</link>
+<joint name="mr_spring_to_body" type="prismatic">
+  <origin xyz="0.051042 -0.35  0.196191" rpy="0 0 0 "/>
+  <parent link="base_link"/>
+  <child link="spring_mr"/>
+  <axis xyz="0.0 0.0 1.0"/>
+  <limit lower="-0.05" upper="0.05" velocity="1.0" effort="10.0" />
+  <dynamics damping="500.0" spring_reference = "0.0" spring_stiffness = "10000.1" friction = "0.75"/>
+</joint>
 <joint name="mrw_to_body" type="continuous">
-  <origin xyz="0.051042 -0.35  0.196191" rpy="0 0 -1.57"/>
-  <parent link="base_link"/>
+  <origin xyz="0.0 0.0 0.0" rpy="0 0 -1.57"/>
+  <parent link="spring_mr"/>
   <child link="mr_wheel_1"/>
   <axis xyz="-1.0 0.0 0.0"/>
 </joint>
+<link name="spring_br">
+  <inertial>
+    <origin xyz="0.0000000000000005 0.00000000000000000005 0.00000000000000000005" rpy="0 0 0"/>
+    <mass value="0.00000000000001"/>
+    <inertia ixx="0.0000006" iyy="0.0000006" izz="0.0000006" ixy="0.0" iyz="0.0" ixz="0.0"/>
+  </inertial>
+  <visual>
+    <origin xyz="0 0 0" rpy="0 0 0"/>
+    <geometry>
+      <box size="0.010 0.010 0.010"/>
+    </geometry>
+    <material name="silver">
+    </material>
+  </visual>
+</link>
+<joint name="br_spring_to_body" type="prismatic">
+  <origin xyz="-0.388958 -0.35  0.196191" rpy="0 0 0 "/>
+  <parent link="base_link"/>
+  <child link="spring_br"/>
+  <axis xyz="0.0 0.0 1.0"/>
+  <limit lower="-0.05" upper="0.05" velocity="1.0" effort="10.0" />
+  <dynamics damping="500.0" spring_reference = "0.0" spring_stiffness = "10000.1" friction = "0.75"/>
+</joint>
 <joint name="brw_to_body" type="continuous">
-  <origin xyz="-0.388958 -0.35  0.196191" rpy="0 0 -1.57"/>
-  <parent link="base_link"/>
+  <origin xyz="0.0 0.0 0.0" rpy="0 0 -1.57"/>
+  <parent link="spring_br"/>
   <child link="br_wheel_1"/>
   <axis xyz="-1.0 0.0 0.0"/>
 </joint>
+<link name="spring_fl">
+  <inertial>
+    <origin xyz="0.0000000000000005 0.00000000000000000005 0.00000000000000000005" rpy="0 0 0"/>
+    <mass value="0.00000000000001"/>
+    <inertia ixx="0.0000006" iyy="0.0000006" izz="0.0000006" ixy="0.0" iyz="0.0" ixz="0.0"/>
+  </inertial>
+  <visual>
+    <origin xyz="0 0 0" rpy="0 0 0"/>
+    <geometry>
+      <box size="0.010 0.010 0.010"/>
+    </geometry>
+    <material name="silver">
+    </material>
+  </visual>
+</link>
+<joint name="fl_spring_to_body" type="prismatic">
+  <origin xyz="0.491042 0.35  0.196191" rpy="0 0 0 "/>
+  <parent link="base_link"/>
+  <child link="spring_fl"/>
+  <axis xyz="0.0 0.0 1.0"/>
+<limit lower="-0.05" upper="0.05" velocity="1.0" effort="10.0" />
+  <dynamics damping="500.0" spring_reference = "0.0" spring_stiffness = "10000.1" friction = "0.75"/>
+</joint>
 <joint name="flw_to_body" type="continuous">
-  <origin xyz="0.491042 0.35  0.196191" rpy="0 0 -1.57"/>
-  <parent link="base_link"/>
+  <origin xyz="0.0 0.0 0.0" rpy="0 0 -1.57"/>
+  <parent link="spring_fl"/>
   <child link="fl_wheel_1"/>
   <axis xyz="-1.0 0.0 0.0"/>
 </joint>
+<link name="spring_ml">
+  <inertial>
+    <origin xyz="0.0000000000000005 0.00000000000000000005 0.00000000000000000005" rpy="0 0 0"/>
+    <mass value="0.00000000000001"/>
+    <inertia ixx="0.0000006" iyy="0.0000006" izz="0.0000006" ixy="0.0" iyz="0.0" ixz="0.0"/>
+  </inertial>
+  <visual>
+    <origin xyz="0 0 0" rpy="0 0 0"/>
+    <geometry>
+      <box size="0.010 0.010 0.010"/>
+    </geometry>
+    <material name="silver">
+    </material>
+  </visual>
+</link>
+<joint name="ml_spring_to_body" type="prismatic">
+  <origin xyz="0.051042 0.35  0.196191" rpy="0 0 0 "/>
+  <parent link="base_link"/>
+  <child link="spring_ml"/>
+  <axis xyz="0.0 0.0 1.0"/>
+<limit lower="-0.05" upper="0.05" velocity="1.0" effort="10.0" />
+  <dynamics damping="500.0" spring_reference = "0.0" spring_stiffness = "10000.1" friction = "0.75"/>
+</joint>
 <joint name="mlw_to_body" type="continuous">
-  <origin xyz="0.051042 0.35  0.196191" rpy="0 0 -1.57"/>
-  <parent link="base_link"/>
+  <origin xyz="0.0 0.0 0.0" rpy="0 0 -1.57"/>
+  <parent link="spring_ml"/>
   <child link="ml_wheel_1"/>
   <axis xyz="-1.0 0.0 0.0"/>
 </joint>
+<link name="spring_bl">
+  <inertial>
+    <origin xyz="0.0000000000000005 0.00000000000000000005 0.00000000000000000005" rpy="0 0 0"/>
+    <mass value="0.00000000000001"/>
+    <inertia ixx="0.0000006" iyy="0.0000006" izz="0.0000006" ixy="0.0" iyz="0.0" ixz="0.0"/>
+  </inertial>
+  <visual>
+    <origin xyz="0 0 0" rpy="0 0 0"/>
+    <geometry>
+      <box size="0.010 0.010 0.010"/>
+    </geometry>
+    <material name="silver">
+    </material>
+  </visual>
+</link>
+<joint name="bl_spring_to_body" type="prismatic">
+  <origin xyz="-0.388958 0.35 0.196191" rpy="0 0 0 "/>
+  <parent link="base_link"/>
+  <child link="spring_bl"/>
+  <axis xyz="0.0 0.0 1.0"/>
+<limit lower="-0.05" upper="0.05" velocity="1.0" effort="10.0" />
+  <dynamics damping="500.0" spring_reference = "0.0" spring_stiffness = "10000.1" friction = "0.75"/>
+</joint>
 <joint name="blw_to_body" type="continuous">
-  <origin xyz="-0.388958 0.35  0.196191" rpy="0 0 -1.57"/>
-  <parent link="base_link"/>
+  <origin xyz="0.0 0.0 0.0" rpy="0 0 -1.57"/>
+  <parent link="spring_bl"/>
   <child link="bl_wheel_1"/>
   <axis xyz="-1.0 0.0 0.0"/>

Commit message: xacro added wheels

File: ros2_ws/src/main/urdf/rover.xacro (robot description, xacro)
@@ -4,4 +4,5 @@
 <xacro:include filename="$(find main)/urdf/Rover.trans" />
 <xacro:include filename="$(find main)/urdf/Rover.gazebo" />
+<xacro:include filename="spring.xacro"/>
 <!-- <link name="dummy_base_link"></link> -->
 <link name="base_link">
@@ -27,128 +28,10 @@
   </collision>
 </link>
-<link name="fr_wheel_1">
-  <inertial>
-    <origin xyz="-0.055000000000000104 1.0988582432869265e-07 -4.0437316894958997e-07" rpy="0 0 0"/>
-    <mass value="11.601995917486711"/>
-    <inertia ixx="0.209416" iyy="0.116407" izz="0.116407" ixy="0.0" iyz="0.0" ixz="-0.0"/>
-  </inertial>
-  <visual>
-    <origin xyz="0.45 0.491042 -0.196191" rpy="0 0 0"/>
-    <geometry>
-      <mesh filename="file://$(find main)/meshes/fr_wheel_1.stl" scale="0.001 0.001 0.001"/>
-    </geometry>
-    <material name="blue">
-      <color rgba="0.1 0.1 0.1 1.0"/>
-    </material>
-  </visual>
-  <collision>
-    <origin xyz="0.45 0.491042 -0.196191" rpy="0 0 0"/>
-    <geometry>
-      <mesh filename="file://$(find main)/meshes/fr_wheel_1.stl" scale="0.001 0.001 0.001"/>
-    </geometry>
-  </collision>
-</link>
-<link name="mr_wheel_1">
-  <inertial>
-    <origin xyz="-0.055000000000000104 1.0988582444665385e-07 -4.0437316886632324e-07" rpy="0 0 0"/>
-    <mass value="11.601995917486711"/>
-    <inertia ixx="0.209416" iyy="0.116407" izz="0.116407" ixy="0.0" iyz="0.0" ixz="-0.0"/>
-  </inertial>
-  <visual>
-    <origin xyz="0.45 0.051042 -0.196191" rpy="0 0 0"/>
-    <geometry>
-      <mesh filename="file://$(find main)/meshes/mr_wheel_1.stl" scale="0.001 0.001 0.001"/>
-    </geometry>
-    <material name="blue">
-      <color rgba="0.1 0.1 0.1 1.0"/>
-    </material>
-  </visual>
-  <collision>
-    <origin xyz="0.45 0.051042 -0.196191" rpy="0 0 0"/>
-    <geometry>
-      <mesh filename="file://$(find main)/meshes/mr_wheel_1.stl" scale="0.001 0.001 0.001"/>
-    </geometry>
-  </collision>
-</link>
-<link name="br_wheel_1">
-  <inertial>
-    <origin xyz="-0.055000000000000104 1.0988582443971495e-07 -4.0437316886632324e-07" rpy="0 0 0"/>
-    <mass value="11.601995917486711"/>
-    <inertia ixx="0.209416" iyy="0.116407" izz="0.116407" ixy="0.0" iyz="0.0" ixz="-0.0"/>
-  </inertial>
-  <visual>
-    <origin xyz="0.45 -0.388958 -0.196191" rpy="0 0 0"/>
-    <geometry>
-      <mesh filename="file://$(find main)/meshes/br_wheel_1.stl" scale="0.001 0.001 0.001"/>
-    </geometry>
-    <material name="blue"/>
-  </visual>
-  <collision>
-    <origin xyz="0.45 -0.388958 -0.196191" rpy="0 0 0"/>
-    <geometry>
-      <mesh filename="file://$(find main)/meshes/br_wheel_1.stl" scale="0.001 0.001 0.001"/>
-    </geometry>
-  </collision>
-</link>
-<link name="fl_wheel_1">
-  <inertial>
-    <origin xyz="0.05500000000000005 1.0988582432869265e-07 -4.0437316894958997e-07" rpy="0 0 0"/>
-    <mass value="11.601995917486711"/>
-    <inertia ixx="0.209416" iyy="0.116407" izz="0.116407" ixy="0.0" iyz="0.0" ixz="-0.0"/>
-  </inertial>
-  <visual>
-    <origin xyz="-0.45 0.491042 -0.196191" rpy="0 0 0"/>
-    <geometry>
-      <mesh filename="file://$(find main)/meshes/fl_wheel_1.stl" scale="0.001 0.001 0.001"/>
-    </geometry>
-    <material name="blue"/>
-  </visual>
-  <collision>
-    <origin xyz="-0.45 0.491042 -0.196191" rpy="0 0 0"/>
-    <geometry>
-      <mesh filename="file://$(find main)/meshes/fl_wheel_1.stl" scale="0.001 0.001 0.001"/>
-    </geometry>
-  </collision>
-</link>
-<link name="ml_wheel_1">
-  <inertial>
-    <origin xyz="0.05500000000000005 1.0988582444665385e-07 -4.0437316886632324e-07" rpy="0 0 0"/>
-    <mass value="11.601995917486711"/>
-    <inertia ixx="0.209416" iyy="0.116407" izz="0.116407" ixy="-0.0" iyz="0.0" ixz="0.0"/>
-  </inertial>
-  <visual>
-    <origin xyz="-0.45 0.051042 -0.196191" rpy="0 0 0"/>
-    <geometry>
-      <mesh filename="file://$(find main)/meshes/ml_wheel_1.stl" scale="0.001 0.001 0.001"/>
-    </geometry>
-    <material name="blue"/>
-  </visual>
-  <collision>
-    <origin xyz="-0.45 0.051042 -0.196191" rpy="0 0 0"/>
-    <geometry>
-      <mesh filename="file://$(find main)/meshes/ml_wheel_1.stl" scale="0.001 0.001 0.001"/>
-    </geometry>
-  </collision>
-</link>
-<link name="bl_wheel_1">
-  <inertial>
-    <origin xyz="0.05500000000000005 1.0988582443971495e-07 -4.0437316886632324e-07" rpy="0 0 0"/>
-    <mass value="11.601995917486711"/>
-    <inertia ixx="0.209416" iyy="0.116407" izz="0.116407" ixy="0.0" iyz="0.0" ixz="0.0"/>
-  </inertial>
-  <visual>
-    <origin xyz="-0.45 -0.388958 -0.196191" rpy="0 0 0"/>
-    <geometry>
-      <mesh filename="file://$(find main)/meshes/bl_wheel_1.stl" scale="0.001 0.001 0.001"/>
-    </geometry>
-    <material name="blue"/>
-  </visual>
-  <collision>
-    <origin xyz="-0.45 -0.388958 -0.196191" rpy="0 0 0"/>
-    <geometry>
-      <mesh filename="file://$(find main)/meshes/bl_wheel_1.stl" scale="0.001 0.001 0.001"/>
-    </geometry>
-  </collision>
-</link>
+<link name="fr_wheel_1"><xacro:wheel/></link>
+<link name="mr_wheel_1"><xacro:wheel/></link>
+<link name="br_wheel_1"><xacro:wheel/></link>
+<link name="fl_wheel_1"><xacro:left_wheel/></link>
+<link name="ml_wheel_1"><xacro:left_wheel/></link>
+<link name="bl_wheel_1"><xacro:left_wheel/></link>
 <link name="cam_link_1">
   <visual>
@@ -170,4 +53,6 @@
     </material>
   </visual>
+</link>
+<link name="rgbd_1">
 </link>
 <gazebo reference="base_link">
@@ -181,11 +66,11 @@
   </sensor>
 </gazebo>
-<gazebo reference="cam_1">
+<gazebo reference="rgbd_1">
   <sensor name="depth_camera" type="depth">
     <always_on>true</always_on>
-    <visualize>true</visualize>
+    <!-- <visualize>true</visualize> -->
     <update_rate>20</update_rate>
     <topic>depth_camera/image</topic>
-    <gz_frame_id>cam_1</gz_frame_id>
+    <gz_frame_id>rgbd_1</gz_frame_id>
     <camera name="depth_camera">
       <camera_info_topic>depth_camera/camera_info</camera_info_topic>
@@ -196,6 +81,27 @@
       </image>
       <clip>
-        <near>0.1</near>
-        <far>5</far>
+        <near>0.5</near>
+        <far>25</far>
+      </clip>
+    </camera>
+  </sensor>
+</gazebo>
+<gazebo reference="cam_1">
+  <sensor name="camera" type="camera">
+    <always_on>true</always_on>
+    <visualize>true</visualize>
+    <update_rate>20</update_rate>
+    <topic>camera/image</topic>
+    <gz_frame_id>cam_1</gz_frame_id>
+    <camera name="camera">
+      <camera_info_topic>camera/camera_info</camera_info_topic>
+      <horizontal_fov>1.8</horizontal_fov>
+      <image>
+        <width>640</width>
+        <height>640</height>
+      </image>
+      <clip>
+        <near>0.5</near>
+        <far>50</far>
       </clip>
     </camera>
@@ -241,17 +147,5 @@
 </joint> -->
 <link name="spring_fr">
-  <inertial>
-    <origin xyz="0.00005 0.00005  0.00005 " rpy="0 0 0"/>
-    <mass value="0.01"/>
-    <inertia ixx="0.0000006" iyy="0.0000006" izz="0.0000006" ixy="0.0" iyz="0.0" ixz="0.0"/>
-  </inertial>
-  <visual>
-    <origin xyz="0 0 0" rpy="0 0 0"/>
-    <geometry>
-      <box size="0.010 0.010 0.010"/>
-    </geometry>
-    <material name="silver">
-    </material>
-  </visual>
+  <xacro:spring_link/>
 </link>
 <joint name="fr_spring_to_body" type="prismatic">
@@ -259,8 +153,6 @@
   <parent link="base_link"/>
   <child link="spring_fr"/>
-  <axis xyz="0.0 0.0 1.0"/>
-  <limit lower="-0.05" upper="0.05" velocity="1.0" effort="10.0" />
-  <dynamics damping="500.0" spring_reference = "0.0" spring_stiffness = "10000.1" friction = "0.75"/>
-</joint>
+  <xacro:spring_joint/>
+  </joint>
 <joint name="frw_to_body" type="continuous">
   <origin xyz="0.0 0.0 0.0" rpy="0 0 -1.57"/>
@@ -270,17 +162,5 @@
 </joint>
 <link name="spring_mr">
-  <inertial>
-    <origin xyz="0.0000000000000005 0.00000000000000000005 0.00000000000000000005" rpy="0 0 0"/>
-    <mass value="0.00000000000001"/>
-    <inertia ixx="0.0000006" iyy="0.0000006" izz="0.0000006" ixy="0.0" iyz="0.0" ixz="0.0"/>
-  </inertial>
-  <visual>
-    <origin xyz="0 0 0" rpy="0 0 0"/>
-    <geometry>
-      <box size="0.010 0.010 0.010"/>
-    </geometry>
-    <material name="silver">
-    </material>
-  </visual>
+  <xacro:spring_link/>
 </link>
 <joint name="mr_spring_to_body" type="prismatic">
@@ -288,7 +168,5 @@
   <parent link="base_link"/>
   <child link="spring_mr"/>
-  <axis xyz="0.0 0.0 1.0"/>
-  <limit lower="-0.05" upper="0.05" velocity="1.0" effort="10.0" />
-  <dynamics damping="500.0" spring_reference = "0.0" spring_stiffness = "10000.1" friction = "0.75"/>
+  <xacro:spring_joint/>
 </joint>
 <joint name="mrw_to_body" type="continuous">
@@ -299,17 +177,5 @@
 </joint>
 <link name="spring_br">
-  <inertial>
-    <origin xyz="0.0000000000000005 0.00000000000000000005 0.00000000000000000005" rpy="0 0 0"/>
-    <mass value="0.00000000000001"/>
-    <inertia ixx="0.0000006" iyy="0.0000006" izz="0.0000006" ixy="0.0" iyz="0.0" ixz="0.0"/>
-  </inertial>
-  <visual>
-    <origin xyz="0 0 0" rpy="0 0 0"/>
-    <geometry>
-      <box size="0.010 0.010 0.010"/>
-    </geometry>
-    <material name="silver">
-    </material>
-  </visual>
+  <xacro:spring_link/>
 </link>
 <joint name="br_spring_to_body" type="prismatic">
@@ -317,7 +183,5 @@
   <parent link="base_link"/>
   <child link="spring_br"/>
-  <axis xyz="0.0 0.0 1.0"/>
-  <limit lower="-0.05" upper="0.05" velocity="1.0" effort="10.0" />
-  <dynamics damping="500.0" spring_reference = "0.0" spring_stiffness = "10000.1" friction = "0.75"/>
+  <xacro:spring_joint/>
 </joint>
 <joint name="brw_to_body" type="continuous">
@@ -328,17 +192,5 @@
 </joint>
 <link name="spring_fl">
-  <inertial>
-    <origin xyz="0.0000000000000005 0.00000000000000000005 0.00000000000000000005" rpy="0 0 0"/>
-    <mass value="0.00000000000001"/>
-    <inertia ixx="0.0000006" iyy="0.0000006" izz="0.0000006" ixy="0.0" iyz="0.0" ixz="0.0"/>
-  </inertial>
-  <visual>
-    <origin xyz="0 0 0" rpy="0 0 0"/>
-    <geometry>
-      <box size="0.010 0.010 0.010"/>
-    </geometry>
-    <material name="silver">
-    </material>
-  </visual>
+  <xacro:spring_link/>
 </link>
 <joint name="fl_spring_to_body" type="prismatic">
@@ -346,7 +198,5 @@
   <parent link="base_link"/>
   <child link="spring_fl"/>
-  <axis xyz="0.0 0.0 1.0"/>
-<limit lower="-0.05" upper="0.05" velocity="1.0" effort="10.0" />
-  <dynamics damping="500.0" spring_reference = "0.0" spring_stiffness = "10000.1" friction = "0.75"/>
+  <xacro:spring_joint/>
 </joint>
 <joint name="flw_to_body" type="continuous">
@@ -357,17 +207,5 @@
 </joint>
 <link name="spring_ml">
-  <inertial>
-    <origin xyz="0.0000000000000005 0.00000000000000000005 0.00000000000000000005" rpy="0 0 0"/>
-    <mass value="0.00000000000001"/>
-    <inertia ixx="0.0000006" iyy="0.0000006" izz="0.0000006" ixy="0.0" iyz="0.0" ixz="0.0"/>
-  </inertial>
-  <visual>
-    <origin xyz="0 0 0" rpy="0 0 0"/>
-    <geometry>
-      <box size="0.010 0.010 0.010"/>
-    </geometry>
-    <material name="silver">
-    </material>
-  </visual>
+  <xacro:spring_link/>
 </link>
 <joint name="ml_spring_to_body" type="prismatic">
@@ -375,7 +213,5 @@
   <parent link="base_link"/>
   <child link="spring_ml"/>
-  <axis xyz="0.0 0.0 1.0"/>
-<limit lower="-0.05" upper="0.05" velocity="1.0" effort="10.0" />
-  <dynamics damping="500.0" spring_reference = "0.0" spring_stiffness = "10000.1" friction = "0.75"/>
+  <xacro:spring_joint/>
 </joint>
 <joint name="mlw_to_body" type="continuous">
@@ -386,17 +222,5 @@
 </joint>
 <link name="spring_bl">
-  <inertial>
-    <origin xyz="0.0000000000000005 0.00000000000000000005 0.00000000000000000005" rpy="0 0 0"/>
-    <mass value="0.00000000000001"/>
-    <inertia ixx="0.0000006" iyy="0.0000006" izz="0.0000006" ixy="0.0" iyz="0.0" ixz="0.0"/>
-  </inertial>
-  <visual>
-    <origin xyz="0 0 0" rpy="0 0 0"/>
-    <geometry>
-      <box size="0.010 0.010 0.010"/>
-    </geometry>
-    <material name="silver">
-    </material>
-  </visual>
+  <xacro:spring_link/>
 </link>
 <joint name="bl_spring_to_body" type="prismatic">
@@ -404,7 +228,5 @@
   <parent link="base_link"/>
   <child link="spring_bl"/>
-  <axis xyz="0.0 0.0 1.0"/>
-<limit lower="-0.05" upper="0.05" velocity="1.0" effort="10.0" />
-  <dynamics damping="500.0" spring_reference = "0.0" spring_stiffness = "10000.1" friction = "0.75"/>
+  <xacro:spring_joint/>
 </joint>
 <joint name="blw_to_body" type="continuous">
@@ -420,7 +242,12 @@
 </joint>
 <joint name="cam_to_camlink" type="fixed">
-  <origin xyz="0 0 0.1" rpy="0 0 0"/>
+  <origin xyz="0 0 0.1" rpy="0 0.60 0"/>
   <parent link="cam_link_1"/>
   <child link="cam_1"/>
 </joint>
+<joint name="rgbd_to_camlink" type="fixed">
+  <origin xyz="0 0 0.1" rpy="0 0.60 0"/>
+  <parent link="cam_link_1"/>
+  <child link="rgbd_1"/>
+</joint>
 </robot>
