Commit message: simple start Makefile + migrate to ROS2 Humble + migrate to Gazebo Classic

File: ros2_ws/src/main/urdf/rover.xacro (robot description, xacro)
@@ -109,5 +109,5 @@
 </gazebo>
 <gazebo reference="base_link">
-  <sensor name="gps" type="navsat">
+  <sensor name="gps" type="gps">
   <always_on>true</always_on>
   <update_rate>20</update_rate>
@@ -154,4 +154,9 @@
   <child link="spring_fr"/>
   <xacro:spring_joint/>
+  <sensor name="force_torque" type="force_torque">
+          <update_rate>30</update_rate>
+          <visualize>true</visualize>
+          <topic>force</topic>
+        </sensor>
   </joint>
 <joint name="frw_to_body" type="continuous">

File: ros2_ws/src/main/urdf/spring.xacro (robot description, xacro)
@@ -17,25 +17,12 @@
     </xacro:macro>
     <xacro:macro name="spring_joint">
-        <axis xyz="0.0 0.0 1.0"/>
-        <limit lower="0.0" upper="0.0" velocity="0.0" effort="1.0" />
-        <!-- <dynamics damping="5000.0" spring_reference ="0.20" spring_stiffness="5000000.0" friction ="0.0"/> -->
-        <!-- <physics> -->
-            <!-- <ode>
-                <implicit_spring_damper>10000</implicit_spring_damper>
-                <cfm_damping>true</cfm_damping>
-                <max_force>5000</max_force>
+        <axis xyz="0.0 0.0 -1.0"/>
+            <limit lower="-0.050" upper="0.050"  velocity="-1.0" effort="-1.0"/>
+            <dynamics damping="50.0" spring_reference ="0.0" spring_stiffness="5.0"/>
+            <ode>
                 <fudge_factor>0.1</fudge_factor>
-                 <cfm>0.0001</cfm>
-                    <erp>0.9</erp>
-                <limit>
-                    <cfm>0.0001</cfm>
-                    <erp>0.9</erp>
-                </limit> -->
-                <!-- <suspension>
-                    <cfm>10000</cfm>
-                    <erp>0.2</erp>
-                </suspension> -->
-            <!-- </ode> -->
-        <!-- </physics> -->
+                <cfm>0.00001</cfm>
+                <erp>0.8</erp>
+            </ode>
     </xacro:macro>
     <xacro:macro name="wheel">

Commit message: container fix

File: ros2_ws/src/main/urdf/rover.xacro (robot description, xacro)
@@ -8,6 +8,6 @@
   <link name="base_link">
     <inertial>
-      <origin xyz="0.0 0.0 0.3" rpy="0 0 -1.57" />
-      <mass value="40.0" />
+      <origin xyz="0.06 0.0 0.3" rpy="0 0 -1.57" />
+      <mass value="20.0" />
       <inertia ixx="11.367893" iyy="2.895706" izz="13.361019" ixy="0.0" iyz="0.0" ixz="0.0" />
     </inertial>
@@ -91,5 +91,5 @@
         </image>
         <clip>
-          <near>0.5</near>
+          <near>0.1</near>
           <far>25</far>
         </clip>
@@ -100,6 +100,6 @@
     <sensor name="camera" type="camera">
       <always_on>true</always_on>
-      <visualize>true</visualize>
-      <update_rate>20</update_rate>
+      <!-- <visualize>true</visualize> -->
+      <update_rate>10</update_rate>
       <topic>camera/image</topic>
       <gz_frame_id>cam_1</gz_frame_id>
@@ -112,6 +112,6 @@
         </image>
         <clip>
-          <near>0.5</near>
-          <far>50</far>
+          <near>0.1</near>
+          <far>25</far>
         </clip>
       </camera>
@@ -121,5 +121,5 @@
     <sensor name="gps" type="gps">
       <always_on>true</always_on>
-      <update_rate>20</update_rate>
+      <update_rate>10</update_rate>
       <visualize>true</visualize>
       <pose>0 0 0 0 0 0</pose>
@@ -193,10 +193,10 @@
   </joint>
   <joint name="camlink_to_body" type="fixed">
-    <origin xyz="0.6 0.0001 0.5" rpy="0 0 0" />
+    <origin xyz="-0.5 0.0 0.8" rpy="0 0 0" />
     <parent link="base_link" />
     <child link="cam_link_1" />
   </joint>
   <joint name="cam_to_camlink" type="fixed">
-    <origin xyz="0 0 0.1" rpy="0 0.60 0" />
+    <origin xyz="0 0 0.1" rpy="0 0.6 0" />
     <parent link="cam_link_1" />
     <child link="cam_1" />

File: ros2_ws/src/main/urdf/spring.xacro (robot description, xacro)
@@ -25,6 +25,6 @@
                     <mu>1</mu>
                     <mu2>1</mu2>
-                    <slip1>0.01</slip1>
-                    <slip2>0.01</slip2>
+                    <slip1>0</slip1>
+                    <slip2>01</slip2>
                 </ode>
             </friction>

Commit message: idk

File: ros2_ws/src/main/urdf/rover.xacro (robot description, xacro)
@@ -9,5 +9,5 @@
     <inertial>
       <origin xyz="0.06 0.0 0.3" rpy="0 0 -1.57" />
-      <mass value="20.0" />
+      <mass value="5.0" />
       <inertia ixx="11.367893" iyy="2.895706" izz="13.361019" ixy="0.0" iyz="0.0" ixz="0.0" />
     </inertial>
@@ -22,5 +22,5 @@
       <origin xyz="0 0 0" rpy="0 0 1.57" />
       <geometry>
-        <mesh filename="file://$(find main)/meshes/base_link.stl" scale="0.001 0.001 0.001" />
+        <!-- <mesh filename="file://$(find main)/meshes/base_link.stl" scale="0.001 0.001 0.001" /> -->
       </geometry>
     </collision>
@@ -43,4 +43,22 @@
   <link name="bl_wheel_1">
     <xacro:left_wheel />
+  </link>
+  <link name="fr_spring">
+    <xacro:spring_link/>
+  </link>
+  <link name="mr_spring">
+    <xacro:spring_link/>
+  </link>
+  <link name="br_spring">
+    <xacro:spring_link/>
+  </link>
+  <link name="fl_spring">
+    <xacro:spring_link/>
+  </link>
+  <link name="ml_spring">
+    <xacro:spring_link/>
+  </link>
+  <link name="bl_spring">
+    <xacro:spring_link/>
   </link>
   <link name="cam_link_1">
@@ -74,4 +92,12 @@
       <child_frame_id>base_link</child_frame_id>
       <topic>imu</topic>
+      <plugin name='imu' filename='libgazebo_ros_imu_sensor.so'>
+        <ros>
+          <!-- <namespace>${mp['namespace']}</namespace> -->
+          <remapping>imu/out:=imu</remapping>
+        </ros>
+        <initial_orientation_as_reference>false</initial_orientation_as_reference>
+        <!-- <frame_name>${mp['namespace']}/base_link</frame_name> -->
+      </plugin>
     </sensor>
   </gazebo>
@@ -124,5 +150,5 @@
       <visualize>true</visualize>
       <pose>0 0 0 0 0 0</pose>
-      <topic>gps</topic>
+      <topic>gps/fix</topic>
       <gz_frame_id>base_link</gz_frame_id>
       <!-- <child_frame_id>base_link</child_frame_id> -->
@@ -143,9 +169,9 @@
         </position_sensing>
       </gps>
-      <!-- <plugin name="my_gps_plugin" filename="libgazebo_ros_gps_sensor.so">
+      <plugin name="gps" filename="libgazebo_ros_gps_sensor.so">
     <ros>
-      <remapping>~/out:=/gps/fix</remapping>
+    <remapping>~/out:=~/fix</remapping>
     </ros>
-  </plugin> -->
+  </plugin>
     </sensor>
   </gazebo>
@@ -156,13 +182,43 @@
   <child link="base_link"/>
 </joint> -->
+  <joint name="fr_spring_to_body" type = "prismatic">
+    <parent link="base_link"/>
+    <child link="fr_spring"/>
+    <xacro:spring_joint/>
+  </joint>
+  <joint name="mr_spring_to_body" type = "prismatic">
+    <parent link="base_link"/>
+    <child link="mr_spring"/>
+    <xacro:spring_joint/>
+  </joint>
+  <joint name="br_spring_to_body" type = "prismatic">
+    <parent link="base_link"/>
+    <child link="br_spring"/>
+    <xacro:spring_joint/>
+  </joint>
+  <joint name="fl_spring_to_body" type = "prismatic">
+    <parent link="base_link"/>
+    <child link="fl_spring"/>
+    <xacro:spring_joint/>
+  </joint>
+  <joint name="ml_spring_to_body" type = "prismatic">
+    <parent link="base_link"/>
+    <child link="ml_spring"/>
+    <xacro:spring_joint/>
+  </joint>
+  <joint name="bl_spring_to_body" type = "prismatic">
+    <parent link="base_link"/>
+    <child link="bl_spring"/>
+    <xacro:spring_joint/>
+  </joint>
   <joint name="frw_to_body" type="continuous">
     <origin xyz="0.491042 -0.35  0.196191" rpy="0 0 -1.57" />
-    <parent link="base_link" />
+    <parent link="fr_spring" />
     <child link="fr_wheel_1" />
     <axis xyz="-1.0 0.0 0.0" />
   </joint>
   <joint name="mrw_to_body" type="continuous">
-    <origin xyz="0.051042 -0.35  0.196191" rpy="0 0 -1.57" />
-    <parent link="base_link" />
+    <origin xyz="0.051042 -0.35  0.19" rpy="0 0 -1.57" />
+    <parent link="mr_spring" />
     <child link="mr_wheel_1" />
     <axis xyz="-1.0 0.0 0.0" />
@@ -170,5 +226,5 @@
   <joint name="brw_to_body" type="continuous">
     <origin xyz="-0.388958 -0.35  0.196191" rpy="0 0 -1.57" />
-    <parent link="base_link" />
+    <parent link="br_spring" />
     <child link="br_wheel_1" />
     <axis xyz="-1.0 0.0 0.0" />
@@ -176,11 +232,11 @@
   <joint name="flw_to_body" type="continuous">
     <origin xyz="0.491042 0.35  0.196191" rpy="0 0 -1.57" />
-    <parent link="base_link" />
+    <parent link="fl_spring" />
     <child link="fl_wheel_1" />
     <axis xyz="-1.0 0.0 0.0" />
   </joint>
   <joint name="mlw_to_body" type="continuous">
-    <origin xyz="0.051042 0.35  0.196191" rpy="0 0 -1.57" />
-    <parent link="base_link" />
+    <origin xyz="0.051042 0.35  0.19" rpy="0 0 -1.57" />
+    <parent link="ml_spring" />
     <child link="ml_wheel_1" />
     <axis xyz="-1.0 0.0 0.0" />
@@ -188,5 +244,5 @@
   <joint name="blw_to_body" type="continuous">
     <origin xyz="-0.388958 0.35 0.196191" rpy="0 0 -1.57" />
-    <parent link="base_link" />
+    <parent link="bl_spring" />
     <child link="bl_wheel_1" />
     <axis xyz="-1.0 0.0 0.0" />

File: ros2_ws/src/main/urdf/spring.xacro (robot description, xacro)
@@ -6,16 +6,19 @@
             <origin xyz="0.0 0.0  0.0 " rpy="0 0 0" />
             <mass value="0.01" />
-            <inertia ixx="0.0" iyy="0.0" izz="0.0" ixy="0.0" iyz="0.0" ixz="0.0" />
+            <inertia ixx="0.01" iyy="0.01" izz="0.01" ixy="0.0" iyz="0.0" ixz="0.0" />
         </inertial>
-        <visual>
+        <!-- <visual>
             <origin xyz="0 0 0" rpy="0 0 0" />
             <geometry>
                 <box size="0.1 0.1 0.1" />
             </geometry>
-        </visual>
+        </visual> -->
     </xacro:macro>
     <xacro:macro name="spring_joint">
-        <axis xyz="0.0 0.0 0.0" />
-        <limit lower="0.0" upper="0.0" velocity="0.0" effort="-1.0" />
+        <axis xyz="0.0 0.0 -1.0" />
+        <limit lower="-0.025" upper="0.025" velocity="-1.0" effort="-1.0" />
+        <dynamics damping="2.0" spring_reference = "10.0" spring_stiffness = "100.1" friction = "0.0"/>
+        <physics>
+        </physics>
     </xacro:macro>
     <xacro:macro name="surface">
@@ -23,15 +26,15 @@
             <friction>
                 <ode>
-                    <mu>1</mu>
-                    <mu2>1</mu2>
-                    <slip1>0</slip1>
-                    <slip2>01</slip2>
+                    <mu>0.95</mu>
+                    <mu2>0.95</mu2>
+                    <slip1>1e-19</slip1>
+                    <slip2>1e-19</slip2>
                 </ode>
             </friction>
             <contact>
                 <ode>
-                    <soft_cfm>0</soft_cfm>
-                    <soft_erp>0.2</soft_erp>
-                    <kp>1e+13</kp>
+                    <cfm>0</cfm>
+                    <erp>0.2</erp>
+                    <kp>200</kp>
                     <kd>1</kd>
                     <max_vel>0.01</max_vel>
@@ -44,5 +47,5 @@
         <inertial>
             <origin xyz="0.05 0 0" rpy="0 1.5707 0" />
-            <mass value="11.6" />
+            <mass value="1.6" />
             <inertia ixx="0.124" ixy="0" ixz="0"
                 iyy="0.124" iyz="0"
@@ -66,5 +69,5 @@
         <inertial>
             <origin xyz="-0.05 0 0" rpy="0 1.5707 3.1415" />
-            <mass value="11.6" />
+            <mass value="1.6" />
             <inertia ixx="0.124" ixy="0" ixz="0"
                 iyy="0.124" iyz="0"

Commit message: betetr physics(bad) + nav2 working

File: ros2_ws/src/main/urdf/rover.xacro (robot description, xacro)
@@ -8,10 +8,10 @@
   <link name="base_link">
     <inertial>
-      <origin xyz="0.06 0.0 0.3" rpy="0 0 -1.57" />
-      <mass value="5.0" />
+      <origin xyz="0.06 0.0 0.3" rpy="0 0 -1.5708" />
+      <mass value="0.10" />
       <inertia ixx="11.367893" iyy="2.895706" izz="13.361019" ixy="0.0" iyz="0.0" ixz="0.0" />
     </inertial>
     <visual>
-      <origin xyz="0 0 0" rpy="0 0 1.57" />
+      <origin xyz="0 0 0" rpy="0 0 1.5708" />
       <geometry>
         <mesh filename="file://$(find main)/meshes/base_link.stl" scale="0.001 0.001 0.001" />
@@ -20,7 +20,7 @@
     </visual>
     <collision>
-      <origin xyz="0 0 0" rpy="0 0 1.57" />
-      <geometry>
-        <!-- <mesh filename="file://$(find main)/meshes/base_link.stl" scale="0.001 0.001 0.001" /> -->
+      <origin xyz="0 0 0.5" rpy="0 0 1.5708" />
+      <geometry>
+        <mesh filename="file://$(find main)/meshes/base_link.stl" scale="0.0001 0.0001 0.0001" />
       </geometry>
     </collision>
@@ -213,5 +213,5 @@
   </joint>
   <joint name="frw_to_body" type="continuous">
-    <origin xyz="0.491042 -0.35  0.196191" rpy="0 0 -1.57" />
+    <origin xyz="0.491042 -0.35  0.196191" rpy="0 0 -1.5708" />
     <parent link="fr_spring" />
     <child link="fr_wheel_1" />
@@ -219,5 +219,5 @@
   </joint>
   <joint name="mrw_to_body" type="continuous">
-    <origin xyz="0.051042 -0.35  0.19" rpy="0 0 -1.57" />
+    <origin xyz="0.051042 -0.35  0.19" rpy="0 0 -1.5708" />
     <parent link="mr_spring" />
     <child link="mr_wheel_1" />
@@ -225,5 +225,5 @@
   </joint>
   <joint name="brw_to_body" type="continuous">
-    <origin xyz="-0.388958 -0.35  0.196191" rpy="0 0 -1.57" />
+    <origin xyz="-0.388958 -0.35  0.196191" rpy="0 0 -1.5708" />
     <parent link="br_spring" />
     <child link="br_wheel_1" />
@@ -231,5 +231,5 @@
   </joint>
   <joint name="flw_to_body" type="continuous">
-    <origin xyz="0.491042 0.35  0.196191" rpy="0 0 -1.57" />
+    <origin xyz="0.491042 0.35  0.196191" rpy="0 0 -1.5708" />
     <parent link="fl_spring" />
     <child link="fl_wheel_1" />
@@ -237,5 +237,5 @@
   </joint>
   <joint name="mlw_to_body" type="continuous">
-    <origin xyz="0.051042 0.35  0.19" rpy="0 0 -1.57" />
+    <origin xyz="0.051042 0.35  0.19" rpy="0 0 -1.5708" />
     <parent link="ml_spring" />
     <child link="ml_wheel_1" />
@@ -243,5 +243,5 @@
   </joint>
   <joint name="blw_to_body" type="continuous">
-    <origin xyz="-0.388958 0.35 0.196191" rpy="0 0 -1.57" />
+    <origin xyz="-0.388958 0.35 0.196191" rpy="0 0 -1.5708" />
     <parent link="bl_spring" />
     <child link="bl_wheel_1" />

File: ros2_ws/src/main/urdf/spring.xacro (robot description, xacro)
@@ -16,9 +16,7 @@
     </xacro:macro>
     <xacro:macro name="spring_joint">
-        <axis xyz="0.0 0.0 -1.0" />
-        <limit lower="-0.025" upper="0.025" velocity="-1.0" effort="-1.0" />
-        <dynamics damping="2.0" spring_reference = "10.0" spring_stiffness = "100.1" friction = "0.0"/>
-        <physics>
-        </physics>
+        <axis xyz="0.0 0.0 1.0" />
+        <limit lower="-0.015" upper="0.015" velocity="-1.0" effort="-1.0" />
+        <dynamics damping="5.0" spring_reference = "0.0" spring_stiffness = "10.1" friction = "0.0"/>
     </xacro:macro>
     <xacro:macro name="surface">
@@ -28,6 +26,6 @@
                     <mu>0.95</mu>
                     <mu2>0.95</mu2>
-                    <slip1>1e-19</slip1>
-                    <slip2>1e-19</slip2>
+                    <slip1>0</slip1>
+                    <slip2>0</slip2>
                 </ode>
             </friction>
@@ -36,8 +34,8 @@
                     <cfm>0</cfm>
                     <erp>0.2</erp>
-                    <kp>200</kp>
+                    <kp>1e8</kp>
                     <kd>1</kd>
                     <max_vel>0.01</max_vel>
-                    <min_depth>0.0</min_depth>
+                    <min_depth>0.00001</min_depth>
                 </ode>
             </contact>
@@ -47,5 +45,5 @@
         <inertial>
             <origin xyz="0.05 0 0" rpy="0 1.5707 0" />
-            <mass value="1.6" />
+            <mass value="40.6" />
             <inertia ixx="0.124" ixy="0" ixz="0"
                 iyy="0.124" iyz="0"
@@ -55,11 +53,10 @@
             <origin xyz="0.05 0 0" rpy="0 1.5707 0" />
             <geometry>
-                <cylinder radius="0.19" length="0.14" />
-            </geometry>
+<xacro:geom/>            </geometry>
         </visual>
         <collision>
             <origin xyz="0.05 0 0" rpy="0 1.5707 0" />
             <geometry>
-                <cylinder radius="0.19" length="0.14" />
+<xacro:geom/>                <!-- <cylinder radius="0.19" length="0.14" /> -->
             </geometry>
             <xacro:surface />
@@ -69,5 +66,5 @@
         <inertial>
             <origin xyz="-0.05 0 0" rpy="0 1.5707 3.1415" />
-            <mass value="1.6" />
+            <mass value="40.6" />
             <inertia ixx="0.124" ixy="0" ixz="0"
                 iyy="0.124" iyz="0"
@@ -77,5 +74,6 @@
             <origin xyz="-0.050 0 0" rpy="0 1.5707 3.1415" />
             <geometry>
-                <cylinder radius="0.19" length="0.14" />
+<xacro:geom/>
+                <!-- <cylinder radius="0.19" length="0.14" /> -->
             </geometry>
             <material name="blue" />
@@ -84,8 +82,12 @@
             <origin xyz="-0.05 0 0" rpy="0 1.57 3.1415" />
             <geometry>
-                <cylinder radius="0.19" length="0.14" />
+                <xacro:geom/>
             </geometry>
             <xacro:surface />
         </collision>
     </xacro:macro>
+    <xacro:macro name="geom">
+    <!-- <cylinder radius="0.19" length="0.14" /> -->
+                <sphere radius="0.19"/>
+    </xacro:macro>
 </robot>
