Commit message: bad nuc

File: ros2_ws/src/simulation/resource/robot.urdf (robot description, URDF)
Before this commit: robot My robot, 0 links, 0 joints
Links:
- added link base_footprint
- added link base_link; visual box size=1.2 0.7 0.2
- added link bl_wheel; visual cylinder length=0.15 radius=0.19
- added link br_wheel; visual cylinder length=0.15 radius=0.19
- added link cam_link; visual box size=0.05 0.1 0.05
- added link fl_wheel; visual cylinder length=0.15 radius=0.19
- added link fr_wheel; visual cylinder length=0.15 radius=0.19
- added link gps
- added link lidar_link; visual box size=0.1 0.1 0.1
- added link ml_wheel; visual cylinder length=0.15 radius=0.19
- added link mr_wheel; visual cylinder length=0.15 radius=0.19
Joints:
- added joint base_link_to_base_footprint: type fixed, parent base_link, child base_footprint, origin xyz=0 0 0 rpy=0 0 0
- added joint base_link_to_bl_wheel: type fixed, parent base_link, child bl_wheel, origin xyz=-0.5 0.5 -0.2 rpy=1.5708 0 0
- added joint base_link_to_br_wheel: type fixed, parent base_link, child br_wheel, origin xyz=-0.5 -0.5 -0.2 rpy=1.5708 0 0
- added joint base_link_to_cam_link: type fixed, parent base_link, child cam_link, origin xyz=0.65 0 0.5 rpy=0 0 0
- added joint base_link_to_fl_wheel: type fixed, parent base_link, child fl_wheel, origin xyz=0.5 0.5 -0.2 rpy=1.5708 0 0
- added joint base_link_to_fr_wheel: type fixed, parent base_link, child fr_wheel, origin xyz=0.5 -0.5 -0.2 rpy=1.5708 0 0
- added joint base_link_to_gps: type fixed, parent base_link, child gps, origin xyz=0 0 0 rpy=0 0 0
- added joint base_link_to_lidar_link: type fixed, parent base_link, child lidar_link, origin xyz=0 0 0.2 rpy=0 0.05 0
- added joint base_link_to_ml_wheel: type fixed, parent base_link, child ml_wheel, origin xyz=0 0.5 -0.2 rpy=1.5708 0 0
- added joint base_link_to_mr_wheel: type fixed, parent base_link, child mr_wheel, origin xyz=0 -0.5 -0.2 rpy=1.5708 0 0
