Commit message: 3d odom

File: ros2_ws/src/main/resource/robot.urdf (robot description, URDF)
Before this commit: robot My robot, 0 links, 0 joints
Links:
- added link base_link; visual box size=1.2 0.7 0.2
- added link fl_wheel; visual cylinder height=0.1 radiuse=0.19
- added link gps
- added link lidar_link; visual box size=0.1 0.1 0.1
Joints:
- added joint base_link_to_fl_wheel: type fixed, parent base_link, child lidar_link, origin xyz=0 0 0 rpy=0 0 0
- added joint base_link_to_gps: type fixed, parent base_link, child gps, origin xyz=0 0 0 rpy=0 0 0
- added joint base_link_to_lidar_link: type fixed, parent base_link, child lidar_link, origin xyz=0 0 0 rpy=0 0 0

Commit message: nav2 params + lidar config

File: ros2_ws/src/main/resource/robot.urdf (robot description, URDF)
Before this commit: robot My robot, 4 links, 3 joints
Links:
- added link bl_wheel; visual cylinder length=0.15 radius=0.19
- added link br_wheel; visual cylinder length=0.15 radius=0.19
- added link fr_wheel; visual cylinder length=0.15 radius=0.19
- added link ml_wheel; visual cylinder length=0.15 radius=0.19
- added link mr_wheel; visual cylinder length=0.15 radius=0.19
- link fl_wheel: geometry visual cylinder length=0.15 radius=0.19
Joints:
- added joint base_link_to_bl_wheel: type fixed, parent base_link, child bl_wheel, origin xyz=-0.5 0.5 -0.2 rpy=1.5708 0 0
- added joint base_link_to_br_wheel: type fixed, parent base_link, child br_wheel, origin xyz=-0.5 -0.5 -0.2 rpy=1.5708 0 0
- added joint base_link_to_fr_wheel: type fixed, parent base_link, child fr_wheel, origin xyz=0.5 -0.5 -0.2 rpy=1.5708 0 0
- added joint base_link_to_ml_wheel: type fixed, parent base_link, child ml_wheel, origin xyz=0 0.5 -0.2 rpy=1.5708 0 0
- added joint base_link_to_mr_wheel: type fixed, parent base_link, child mr_wheel, origin xyz=0 -0.5 -0.2 rpy=1.5708 0 0
- joint base_link_to_fl_wheel: child lidar_link -> fl_wheel; origin xyz=0 0 0 rpy=0 0 0 -> xyz=0.5 0.5 -0.2 rpy=1.5708 0 0
- joint base_link_to_lidar_link: origin xyz=0 0 0 rpy=0 0 0 -> xyz=0 0 0.2 rpy=0 0.05 0

Commit message: scan filter node

File: ros2_ws/src/main/resource/robot.urdf (robot description, URDF)
Before this commit: robot My robot, 9 links, 8 joints
Links:
- added link cam_link; visual box size=0.05 0.1 0.05
Joints:
- added joint base_link_to_cam_link: type fixed, parent base_link, child cam_link, origin xyz=0.65 0 0 rpy=0 0 0

Commit message: navigation+map improved+ GPS functionality

File: ros2_ws/src/main/resource/robot.urdf (robot description, URDF)
Before this commit: robot My robot, 10 links, 9 joints
Links:
- added link base_footprint
Joints:
- added joint base_link_to_base_footprint: type fixed, parent base_link, child base_footprint, origin xyz=0 0 0 rpy=0 0 0
- joint base_link_to_cam_link: origin xyz=0.65 0 0 rpy=0 0 0 -> xyz=0.65 0 0.5 rpy=0 0 0

Commit message: urdf working

File: ros2_ws/src/main/resource/robot.urdf (robot description, URDF)
Before this commit: robot My robot, 11 links, 10 joints
Links:
- added link rs1_link; visual box size=0.05 0.1 0.05
- added link rs2_link; visual box size=0.05 0.1 0.05
Joints:
- added joint cam_link_to_rs1_link: type fixed, parent cam_link, child rs1_link, origin xyz=0 0.07 0 rpy=3.1415 0 0.7
- added joint cam_link_to_rs2_link: type fixed, parent cam_link, child rs2_link, origin xyz=0 -0.07 0 rpy=0 0 -0.7
- joint base_link_to_cam_link: origin xyz=0.65 0 0.5 rpy=0 0 0 -> xyz=0.65 0 0.5 rpy=3.1415 0 0
- joint base_link_to_lidar_link: origin xyz=0 0 0.2 rpy=0 0.05 0 -> xyz=0.65 0 0.5 rpy=0 0.05 3.1415

Commit message: yolo working beta

File: ros2_ws/src/main/resource/robot.urdf (robot description, URDF)
Before this commit: robot My robot, 13 links, 12 joints
Joints:
- joint base_link_to_cam_link: origin xyz=0.65 0 0.5 rpy=3.1415 0 0 -> xyz=0.65 0 0.5 rpy=0 0 0
- joint base_link_to_lidar_link: origin xyz=0.65 0 0.5 rpy=0 0.05 3.1415 -> xyz=0.65 0 0.5 rpy=0 -0.05 3.1415
- joint cam_link_to_rs1_link: origin xyz=0 0.07 0 rpy=3.1415 0 0.7 -> xyz=0 0.07 0 rpy=0 0 0.5
- joint cam_link_to_rs2_link: origin xyz=0 -0.07 0 rpy=0 0 -0.7 -> xyz=0 -0.07 0 rpy=0 0 -0.5

Commit message: uart wroten

File: ros2_ws/src/main/resource/robot.urdf (robot description, URDF)
Before this commit: robot My robot, 11 links, 10 joints
Links:
- added link imu1_link, mass 0.01; collision box size=0.05 0.05 0.05
- link ml_wheel: mass None -> 0.01; geometry collision box size=0.05 0.05 0.05; visual cylinder length=0.15 radius=0.19
Joints:
- added joint imu1_joint: type fixed, parent base_link, child imu1_link, origin xyz=0.5 0 0.1 rpy=0 0 0

Commit message: imu node working

File: ros2_ws/src/main/resource/robot.urdf (robot description, URDF)
Before this commit: robot My robot, 13 links, 12 joints
Links:
- added link mount_link; visual box size=0.02 0.03 0.16
- link bl_wheel: geometry visual cylinder length=0.15 radius=0.17
- link br_wheel: geometry visual cylinder length=0.15 radius=0.17
- link fl_wheel: geometry visual cylinder length=0.15 radius=0.17
- link fr_wheel: geometry visual cylinder length=0.15 radius=0.17
- link gps: geometry visual box size=0.05 0.05 0.05
- link lidar_link: geometry visual box size=0.05 0.05 0.05
- link ml_wheel: geometry visual cylinder length=0.15 radius=0.17
- link mr_wheel: geometry visual cylinder length=0.15 radius=0.17
Joints:
- removed joint base_link_to_cam_link
- removed joint base_link_to_gps
- removed joint base_link_to_lidar_link
- added joint base_link_to_mount_link: type fixed, parent base_link, child mount_link, origin xyz=0.56 0 0.2 rpy=0 0 0
- added joint mount_link_to_cam_link: type fixed, parent mount_link, child cam_link, origin xyz=0 0 -0.05 rpy=0 0 0
- added joint mount_link_to_gps: type fixed, parent base_link, child gps, origin xyz=0.155 0 0 rpy=0 0 0
- added joint mount_link_to_lidar_link: type fixed, parent mount_link, child lidar_link, origin xyz=0.0 0 0.1 rpy=0 -0.05 0

Commit message: speed + state + indicators + joy

File: ros2_ws/src/main/resource/robot.urdf (robot description, URDF)
Before this commit: robot My robot, 14 links, 13 joints
Joints:
- joint base_link_to_mount_link: origin xyz=0.56 0 0.2 rpy=0 0 0 -> xyz=0.535 0 0.2 rpy=0 0 0
- joint mount_link_to_lidar_link: origin xyz=0.0 0 0.1 rpy=0 -0.05 0 -> xyz=0.0 0 0.1 rpy=0 -0.05 3.1415
